File: hardware/DesignLab.kicad_sch (KiCad schematic)
At the start: 87 parts

Commit message: PCB design proposal
Parts:
- SW14, SW3: manf# EVQ-PLFA08 -> TL3342F450QG
Changed lines of the file:
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@@
       (effects (font (size 1.27 1.27)) hide)
     )
-    (property "manf#" "EVQ-PLFA08" (id 5) (at 39.116 217.424 0)
+    (property "manf#" "TL3342F450QG" (id 5) (at 39.116 217.424 0)
       (effects (font (size 1.27 1.27)) hide)
     )
@@
       (effects (font (size 1.27 1.27)) hide)
     )
-    (property "manf#" "EVQ-PLFA08" (id 5) (at 95.758 266.954 0)
+    (property "manf#" "TL3342F450QG" (id 5) (at 95.758 266.954 0)
       (effects (font (size 1.27 1.27)) hide)
     )
@@
     )
     (path "/3e6a15bc-a0c3-47bb-beab-64d542edcc16"
-      (reference "SW3") (unit 1) (value "Button") (footprint "Design:EVQPLFA08")
+      (reference "SW3") (unit 1) (value "REC") (footprint "Button_Switch_SMD:SW_SPST_TL3342")
     )
     (path "/04f33ebb-60dd-456c-8657-ff17e4842fa1"
@@
     )
     (path "/e348a61a-40cc-454f-a7fc-2d69f7f1dd26"
-      (reference "SW14") (unit 1) (value "Button") (footprint "Design:EVQPLFA08")
+      (reference "SW14") (unit 1) (value "VOL") (footprint "Button_Switch_SMD:SW_SPST_TL3342")
     )
     (path "/966b56d4-3c92-4a21-bfbb-4f71bc45350f"

Commit message: Corrected BOM
Parts:
- BZ1: provedor (none) -> MOUSER
- C1, C3: manf# CL10C270JB8NNNC -> C0603C270J5GAC7411
- D2: LCSC# (none) -> C118339; Stock en EC (none) -> Yes; provedor (none) -> LCSC
- J1: manf# (none) -> OS102011MA1QN1; provedor (none) -> MOUSER
- J2: Stock en EC (none) -> Yes
- P1, Q1, SW12, SW14, SW15, SW3: Stock en EC No -> Yes
- R20: LCSC# (none) -> C279996; Stock en EC (none) -> Yes; provedor (none) -> LCSC
- SW1, SW2: manf# (none) -> OS102011MS2QN1
- SW13: manf# (none) -> OS102011MA1QN1
- U2: manf# RP2040-7-500 -> 358-RP2040CHIP-7-500
Changed lines of the file:
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@@
       (effects (font (size 1.27 1.27)) hide)
     )
-    (property "manf#" "CL10C270JB8NNNC" (id 5) (at 33.274 98.552 0)
+    (property "manf#" "C0603C270J5GAC7411" (id 5) (at 33.274 98.552 0)
       (effects (font (size 1.27 1.27)) hide)
     )
@@
       (effects (font (size 1.27 1.27)) hide)
     )
-    (property "Stock en EC" "No" (id 7) (at 371.475 44.323 0)
+    (property "Stock en EC" "Yes" (id 7) (at 371.475 44.323 0)
       (effects (font (size 1.27 1.27)) hide)
     )
@@
       (effects (font (size 1.27 1.27)) hide)
     )
+    (property "LCSC#" " C279996" (id 4) (at 151.384 132.715 0)
+      (effects (font (size 1.27 1.27)) hide)
+    )
+    (property "provedor" "LCSC" (id 5) (at 151.384 132.715 0)
+      (effects (font (size 1.27 1.27)) hide)
+    )
+    (property "Stock en EC" "Yes" (id 6) (at 151.384 132.715 0)
+      (effects (font (size 1.27 1.27)) hide)
+    )
     (pin "1")
     (pin "2")
@@
       (effects (font (size 1.27 1.27)) hide)
     )
+    (property "LCSC#" "C118339" (id 4) (at 159.512 132.715 0)
+      (effects (font (size 1.27 1.27)) hide)
+    )
+    (property "Stock en EC" "Yes" (id 5) (at 159.512 132.715 0)
+      (effects (font (size 1.27 1.27)) hide)
+    )
+    (property "provedor" "LCSC" (id 6) (at 159.512 132.715 0)
+      (effects (font (size 1.27 1.27)) hide)
+    )
     (pin "1")
     (pin "2")
@@
       (effects (font (size 1.27 1.27)) hide)
     )
-    (property "Stock en EC" "No" (id 7) (at 39.116 217.424 0)
+    (property "Stock en EC" "Yes" (id 7) (at 39.116 217.424 0)
       (effects (font (size 1.27 1.27)) hide)
     )
@@
       (effects (font (size 1.27 1.27)) hide)
     )
-    (property "manf#" "" (id 5) (at 37.846 242.062 0)
+    (property "manf#" "OS102011MS2QN1" (id 5) (at 37.846 242.062 0)
       (effects (font (size 1.27 1.27)) hide)
     )
@@
       (effects (font (size 1.27 1.27)) hide)
     )
-    (property "Stock en EC" "No" (id 6) (at 169.926 43.688 0)
+    (property "Stock en EC" "Yes" (id 6) (at 169.926 43.688 0)
       (effects (font (size 1.27 1.27)) hide)
     )
@@
       (effects (font (size 1.27 1.27)) hide)
     )
+    (property "provedor" "MOUSER" (id 6) (at 365.379 109.728 0)
+      (effects (font (size 1.27 1.27)) hide)
+    )
     (pin "1")
     (pin "2")
@@
       (effects (font (size 1.27 1.27)) hide)
     )
-    (property "Stock en EC" "No" (id 6) (at 166.751 22.987 0)
+    (property "Stock en EC" "Yes" (id 6) (at 166.751 22.987 0)
       (effects (font (size 1.27 1.27)) hide)
     )
@@
       (effects (font (size 1.27 1.27)) hide)
     )
-    (property "manf#" "RP2040-7-500" (id 5) (at 79.629 81.153 0)
+    (property "manf#" "358-RP2040CHIP-7-500" (id 5) (at 79.629 81.153 0)
       (effects (font (size 1.27 1.27)) hide)
     )
@@
       (effects (font (size 1.27 1.27)) hide)
     )
-    (property "manf#" "CL10C270JB8NNNC" (id 5) (at 20.574 97.917 0)
+    (property "manf#" "C0603C270J5GAC7411" (id 5) (at 20.574 97.917 0)
       (effects (font (size 1.27 1.27)) hide)
     )
@@
       (effects (font (size 1.27 1.27)) hide)
     )
-    (property "Stock en EC" "No" (id 7) (at 315.468 168.656 0)
+    (property "Stock en EC" "Yes" (id 7) (at 315.468 168.656 0)
       (effects (font (size 1.27 1.27)) hide)
     )
@@
       (effects (font (size 1.27 1.27)) hide)
     )
-    (property "manf#" "" (id 5) (at 324.993 175.006 0)
+    (property "manf#" "OS102011MA1QN1" (id 5) (at 324.993 175.006 0)
       (effects (font (size 1.27 1.27)) hide)
     )
@@
       (effects (font (size 1.27 1.27)) hide)
     )
+    (property "manf#" "OS102011MA1QN1" (id 5) (at 254.381 50.038 0)
+      (effects (font (size 1.27 1.27)) hide)
+    )
+    (property "provedor" "MOUSER" (id 6) (at 254.381 50.038 0)
+      (effects (font (size 1.27 1.27)) hide)
+    )
     (pin "1")
     (pin "10")
@@
       (effects (font (size 1.27 1.27)) hide)
     )
-    (property "manf#" "" (id 5) (at 36.576 266.954 0)
+    (property "manf#" "OS102011MS2QN1" (id 5) (at 36.576 266.954 0)
       (effects (font (size 1.27 1.27)) hide)
     )
@@
       (effects (font (size 1.27 1.27)) hide)
     )
+    (property "Stock en EC" "Yes" (id 4) (at 356.108 227.203 0)
+      (effects (font (size 1.27 1.27)) hide)
+    )
     (pin "1")
     (pin "2")
@@
       (effects (font (size 1.27 1.27)) hide)
     )
-    (property "Stock en EC" "No" (id 7) (at 95.758 266.954 0)
+    (property "Stock en EC" "Yes" (id 7) (at 95.758 266.954 0)
       (effects (font (size 1.27 1.27)) hide)
     )
