File: hardware/DesignLab.kicad_sch (KiCad schematic)
At the start: 83 parts

Commit message: Fix pin EN_SOUND
Parts:
- BT4: value (none) -> Battery_Cell; footprint (none) -> Connector_PinHeader_2.54mm:PinHeader_1x02_P2.54mm_Vertical
- BZ1: value (none) -> Buzzer; footprint (none) -> Connector_PinHeader_2.54mm:PinHeader_1x02_P2.54mm_Vertical
- C1, C3: value (none) -> 27pF; footprint (none) -> Capacitor_SMD:C_0603_1608Metric
- C10, C11, C12, C13, C14, C15, C16, C5, C6, C8, C9: value (none) -> 100nF; footprint (none) -> Capacitor_SMD:C_0402_1005Metric_Pad0.74x0.62mm_HandSolder
- C2: value (none) -> 0.1uF; footprint (none) -> Capacitor_SMD:C_0402_1005Metric_Pad0.74x0.62mm_HandSolder
- C20: value (none) -> 47uF; footprint (none) -> Capacitor_SMD:C_0603_1608Metric
- C21, C22, C4, C7: value (none) -> 1uF; footprint (none) -> Capacitor_SMD:C_0603_1608Metric
- C23, C24: value (none) -> 220pF; footprint (none) -> Capacitor_SMD:C_0603_1608Metric
- C25, C26, C27: value (none) -> 10uF; footprint (none) -> Capacitor_SMD:C_0402_1005Metric_Pad0.74x0.62mm_HandSolder
- C29: value (none) -> 100nF; footprint (none) -> Capacitor_SMD:C_0402_1005Metric
- D1: value (none) -> MBR120; footprint (none) -> Design:SODFL3616X98N
- D2: value (none) -> LED; footprint (none) -> Capacitor_SMD:C_0603_1608Metric
- F1: value (none) -> 0.5A; footprint (none) -> Fuse:Fuse_0805_2012Metric
- J1: value (none) -> Micro_SD_Card_Det; footprint (none) -> Design:1140084168
- J2: value (none) -> Conn_01x04_Female; footprint (none) -> Connector_PinHeader_2.54mm:PinHeader_1x04_P2.54mm_Vertical
- P1: value (none) -> USB_C_Plug_USB2.0; footprint (none) -> Connectors:C393939
- Q1: value (none) -> DMG3415U-7; footprint (none) -> Package_TO_SOT_SMD:SOT-23
- R1: value (none) -> 1K; footprint (none) -> Resistor_SMD:R_0603_1608Metric
- R10, R11, R12, R22: value (none) -> 10K; footprint (none) -> Capacitor_SMD:C_0603_1608Metric
- R13: value (none) -> 1.8K; footprint (none) -> Resistor_SMD:R_0603_1608Metric
- R14, R15, R9: value (none) -> 100; footprint (none) -> Resistor_SMD:R_0603_1608Metric
- R16: value (none) -> 10K; footprint (none) -> Resistor_SMD:R_0603_1608Metric
- R17, R23: value (none) -> 100K; footprint (none) -> Resistor_SMD:R_0603_1608Metric
- R18, R19: value (none) -> 5k1; footprint (none) -> Resistor_SMD:R_0603_1608Metric
- R2, R3: value (none) -> 27; footprint (none) -> Resistor_SMD:R_0603_1608Metric
- R20: value (none) -> 330; footprint (none) -> Resistor_SMD:R_0603_1608Metric
- R21, R4, R6, R7: value (none) -> 100; footprint (none) -> Capacitor_SMD:C_0603_1608Metric
- R5: value (none) -> 4K7; footprint (none) -> Resistor_SMD:R_0603_1608Metric
- R8: value (none) -> 220; footprint (none) -> Resistor_SMD:R_0603_1608Metric
- SW1: value (none) -> SW_DPDT_x2; footprint (none) -> Design:OS102011MA1QN1
- SW10, SW11, SW4, SW5, SW6, SW7, SW8, SW9: value (none) -> Button; footprint (none) -> Design:EVQPLFA08
- SW12: value (none) -> RESET; footprint (none) -> Button_Switch_SMD:SW_SPST_TL3342
- SW13: value (none) -> ON; footprint (none) -> Design:OS102011MA1QN1
- SW14: value (none) -> VOL; footprint (none) -> Button_Switch_SMD:SW_SPST_TL3342
- SW15: value (none) -> BOOT; footprint (none) -> Button_Switch_SMD:SW_SPST_TL3342
- SW3: value (none) -> REC; footprint (none) -> Button_Switch_SMD:SW_SPST_TL3342
- U1: value (none) -> SPH0641LM4H; footprint (none) -> Sensors:MIC_SPH0641LM4H-1
- U10: value (none) -> MCP4018-xxxxLT; footprint (none) -> Design:SOT65P210X110-6N
- U2: value (none) -> RP2040; footprint (none) -> badge_pwnCon:RP2040-QFN-56
- U3, U4, U5, U9: value (none) -> QRE1113; footprint (none) -> Design:QRE1113
- U6: value (none) -> W25Q80DVSSIG; footprint (none) -> Design:SOIC127P798X216-8N
- U7: value (none) -> PAM8302AASCR; footprint (none) -> Package_SO:MSOP-8_3x3mm_P0.65mm
- U8: value (none) -> AP2112K-3.3; footprint (none) -> Package_TO_SOT_SMD:SOT-23-5
- Y1: value (none) -> 12Mhz; footprint (none) -> Crystal:Crystal_SMD_HC49-SD
- sw2: value (none) -> SW_DPDT_x2; footprint (none) -> Design:7829H-1-051LF
Connections:
- net SD is gone; now on net EN_SOUND: R16.1, U7.1 (~{SD})

Commit message: Buttons were changed, routed and assigned another pin
Parts:
- removed SW10, SW11, SW4, SW5, SW6, SW7, SW8, SW9: Button, Design:EVQPLFA08, symbol EVQ-PLFA08:EVQ-PLFA08
- removed sw2: SW_DPDT_x2, Design:7829H-1-051LF, symbol Switch:SW_DPDT_x2
- added SW10, SW2, SW4, SW5, SW6, SW7, SW8, SW9: (no value), symbol Switch:SW_Push
- added SW11: (no value), symbol Switch:SW_DPDT_x2
- BT4: value Battery_Cell -> (none); footprint Connector_PinHeader_2.54mm:PinHeader_1x02_P2.54mm_Vertical -> (none)
- BZ1: value Buzzer -> (none); footprint Connector_PinHeader_2.54mm:PinHeader_1x02_P2.54mm_Vertical -> (none)
- C1, C3: value 27pF -> (none); footprint Capacitor_SMD:C_0603_1608Metric -> (none)
- C10, C11, C12, C13, C14, C15, C16, C5, C6, C8, C9: value 100nF -> (none); footprint Capacitor_SMD:C_0402_1005Metric_Pad0.74x0.62mm_HandSolder -> (none)
- C2: value 0.1uF -> (none); footprint Capacitor_SMD:C_0402_1005Metric_Pad0.74x0.62mm_HandSolder -> (none)
- C20: value 47uF -> (none); footprint Capacitor_SMD:C_0603_1608Metric -> (none)
- C21, C22, C4, C7: value 1uF -> (none); footprint Capacitor_SMD:C_0603_1608Metric -> (none)
- C23, C24: value 220pF -> (none); footprint Capacitor_SMD:C_0603_1608Metric -> (none)
- C25, C26, C27: value 10uF -> (none); footprint Capacitor_SMD:C_0402_1005Metric_Pad0.74x0.62mm_HandSolder -> (none)
- C29: value 100nF -> (none); footprint Capacitor_SMD:C_0402_1005Metric -> (none)
- D1: value MBR120 -> (none); footprint Design:SODFL3616X98N -> (none)
- D2: value LED -> (none); footprint Capacitor_SMD:C_0603_1608Metric -> (none)
- F1: value 0.5A -> (none); footprint Fuse:Fuse_0805_2012Metric -> (none)
- J1: value Micro_SD_Card_Det -> (none); footprint Design:1140084168 -> (none)
- J2: value Conn_01x04_Female -> (none); footprint Connector_PinHeader_2.54mm:PinHeader_1x04_P2.54mm_Vertical -> (none)
- P1: value USB_C_Plug_USB2.0 -> (none); footprint Connectors:C393939 -> (none)
- Q1: value DMG3415U-7 -> (none); footprint Package_TO_SOT_SMD:SOT-23 -> (none)
- R1: value 1K -> (none); footprint Resistor_SMD:R_0603_1608Metric -> (none)
- R10, R11, R12, R22: value 10K -> (none); footprint Capacitor_SMD:C_0603_1608Metric -> (none)
- R13: value 1.8K -> (none); footprint Resistor_SMD:R_0603_1608Metric -> (none)
- R14, R15, R9: value 100 -> (none); footprint Resistor_SMD:R_0603_1608Metric -> (none)
- R16: value 10K -> (none); footprint Resistor_SMD:R_0603_1608Metric -> (none)
- R17, R23: value 100K -> (none); footprint Resistor_SMD:R_0603_1608Metric -> (none)
- R18, R19: value 5k1 -> (none); footprint Resistor_SMD:R_0603_1608Metric -> (none)
- R2, R3: value 27 -> (none); footprint Resistor_SMD:R_0603_1608Metric -> (none)
- R20: value 330 -> (none); footprint Resistor_SMD:R_0603_1608Metric -> (none)
- R21, R4, R6, R7: value 100 -> (none); footprint Capacitor_SMD:C_0603_1608Metric -> (none)
- R5: value 4K7 -> (none); footprint Resistor_SMD:R_0603_1608Metric -> (none)
- R8: value 220 -> (none); footprint Resistor_SMD:R_0603_1608Metric -> (none)
- SW1: value SW_DPDT_x2 -> (none); footprint Design:OS102011MA1QN1 -> (none)
- SW12: value RESET -> (none); footprint Button_Switch_SMD:SW_SPST_TL3342 -> (none)
- SW13: value ON -> (none); footprint Design:OS102011MA1QN1 -> (none)
- SW14: value VOL -> (none); footprint Button_Switch_SMD:SW_SPST_TL3342 -> (none)
- SW15: value BOOT -> (none); footprint Button_Switch_SMD:SW_SPST_TL3342 -> (none)
- SW3: value REC -> (none); footprint Button_Switch_SMD:SW_SPST_TL3342 -> (none)
- U1: value SPH0641LM4H -> (none); footprint Sensors:MIC_SPH0641LM4H-1 -> (none)
- U10: value MCP4018-xxxxLT -> (none); footprint Design:SOT65P210X110-6N -> (none)
- U2: value RP2040 -> (none); footprint badge_pwnCon:RP2040-QFN-56 -> (none)
- U3, U4, U5, U9: value QRE1113 -> (none); footprint Design:QRE1113 -> (none)
- U6: value W25Q80DVSSIG -> (none); footprint Design:SOIC127P798X216-8N -> (none)
- U7: value PAM8302AASCR -> (none); footprint Package_SO:MSOP-8_3x3mm_P0.65mm -> (none)
- U8: value AP2112K-3.3 -> (none); footprint Package_TO_SOT_SMD:SOT-23-5 -> (none)
- Y1: value 12Mhz -> (none); footprint Crystal:Crystal_SMD_HC49-SD -> (none)
Connections:
- net +3V3: now also SW11.1 (A)
- net D0: now also U2.15 (GPIO12), SW5.2; no longer U2.13 (GPIO10)
- net D1: now also SW6.2
- net D2: now also U2.11 (GPIO8), SW8.2; no longer U2.15 (GPIO12)
- net D3: now also SW4.2
- net D4: now also U2.12 (GPIO9), SW10.2; no longer U2.4 (GPIO2)
- net D5: now also U2.31 (GPIO20), SW2.2; no longer U2.11 (GPIO8)
- net D6: now also U2.13 (GPIO10), SW7.2; no longer U2.12 (GPIO9)
- net D7: now also U2.4 (GPIO2), SW9.2; no longer U2.31 (GPIO20)
- net GND: now also SW10.1, SW11.3 (C), SW2.1, SW4.1, SW5.1, SW6.1, SW7.1, SW8.1, SW9.1
- net LANG: now also SW11.2 (B)

Commit message: Rounded PCB and added new labels
Parts:
- BT4: value (none) -> Battery_Cell; footprint (none) -> Connector_PinHeader_2.54mm:PinHeader_1x02_P2.54mm_Vertical
- BZ1: value (none) -> Buzzer; footprint (none) -> Connector_PinHeader_2.54mm:PinHeader_1x02_P2.54mm_Vertical
- C1, C3: value (none) -> 27pF; footprint (none) -> Capacitor_SMD:C_0603_1608Metric
- C10, C11, C12, C13, C14, C15, C16, C5, C6, C8, C9: value (none) -> 100nF; footprint (none) -> Capacitor_SMD:C_0402_1005Metric_Pad0.74x0.62mm_HandSolder
- C2: value (none) -> 0.1uF; footprint (none) -> Capacitor_SMD:C_0402_1005Metric_Pad0.74x0.62mm_HandSolder
- C20: value (none) -> 47uF; footprint (none) -> Capacitor_SMD:C_0603_1608Metric
- C21, C22, C4, C7: value (none) -> 1uF; footprint (none) -> Capacitor_SMD:C_0603_1608Metric
- C23, C24: value (none) -> 220pF; footprint (none) -> Capacitor_SMD:C_0603_1608Metric
- C25, C26, C27: value (none) -> 10uF; footprint (none) -> Capacitor_SMD:C_0402_1005Metric_Pad0.74x0.62mm_HandSolder
- C29: value (none) -> 100nF; footprint (none) -> Capacitor_SMD:C_0402_1005Metric
- D1: value (none) -> MBR120; footprint (none) -> Design:SODFL3616X98N
- D2: value (none) -> LED; footprint (none) -> Capacitor_SMD:C_0603_1608Metric
- F1: value (none) -> 0.5A; footprint (none) -> Fuse:Fuse_0805_2012Metric
- J1: value (none) -> Micro_SD_Card_Det; footprint (none) -> Design:1140084168
- J2: value (none) -> Conn_01x04_Female; footprint (none) -> Connector_PinHeader_2.54mm:PinHeader_1x04_P2.54mm_Vertical
- P1: value (none) -> USB_C_Plug_USB2.0; footprint (none) -> Connectors:C393939
- Q1: value (none) -> DMG3415U-7; footprint (none) -> Package_TO_SOT_SMD:SOT-23
- R1: value (none) -> 1K; footprint (none) -> Resistor_SMD:R_0603_1608Metric
- R10, R11, R12, R22: value (none) -> 10K; footprint (none) -> Capacitor_SMD:C_0603_1608Metric
- R13: value (none) -> 1.8K; footprint (none) -> Resistor_SMD:R_0603_1608Metric
- R14, R15, R9: value (none) -> 100; footprint (none) -> Resistor_SMD:R_0603_1608Metric
- R16: value (none) -> 10K; footprint (none) -> Resistor_SMD:R_0603_1608Metric
- R17, R23: value (none) -> 100K; footprint (none) -> Resistor_SMD:R_0603_1608Metric
- R18, R19: value (none) -> 5k1; footprint (none) -> Resistor_SMD:R_0603_1608Metric
- R2, R3: value (none) -> 27; footprint (none) -> Resistor_SMD:R_0603_1608Metric
- R20: value (none) -> 330; footprint (none) -> Resistor_SMD:R_0603_1608Metric
- R21, R4, R6, R7: value (none) -> 100; footprint (none) -> Capacitor_SMD:C_0603_1608Metric
- R5: value (none) -> 4K7; footprint (none) -> Resistor_SMD:R_0603_1608Metric
- R8: value (none) -> 220; footprint (none) -> Resistor_SMD:R_0603_1608Metric
- SW1: value (none) -> SW_DPDT_x2; footprint (none) -> Design:OS102011MA1QN1
- SW10, SW2, SW4, SW5, SW6, SW7, SW8, SW9: value (none) -> SW_Push; footprint (none) -> Design:Button
- SW11: value (none) -> SW_DPDT_x2; footprint (none) -> Design:7829H-1-051LF
- SW12: value (none) -> RESET; footprint (none) -> Button_Switch_SMD:SW_SPST_TL3342
- SW13: value (none) -> ON; footprint (none) -> Design:OS102011MA1QN1
- SW14: value (none) -> VOL; footprint (none) -> Button_Switch_SMD:SW_SPST_TL3342
- SW15: value (none) -> BOOT; footprint (none) -> Button_Switch_SMD:SW_SPST_TL3342
- SW3: value (none) -> REC; footprint (none) -> Button_Switch_SMD:SW_SPST_TL3342
- U1: value (none) -> SPH0641LM4H; footprint (none) -> Sensors:MIC_SPH0641LM4H-1
- U10: value (none) -> MCP4018-xxxxLT; footprint (none) -> Design:SOT65P210X110-6N
- U2: value (none) -> RP2040; footprint (none) -> badge_pwnCon:RP2040-QFN-56
- U3, U4, U5, U9: value (none) -> QRE1113; footprint (none) -> Design:QRE1113
- U6: value (none) -> W25Q80DVSSIG; footprint (none) -> Design:SOIC127P798X216-8N
- U7: value (none) -> PAM8302AASCR; footprint (none) -> Package_SO:MSOP-8_3x3mm_P0.65mm
- U8: value (none) -> AP2112K-3.3; footprint (none) -> Package_TO_SOT_SMD:SOT-23-5
- Y1: value (none) -> 12Mhz; footprint (none) -> Crystal:Crystal_SMD_HC49-SD
Connections:
- net S2: now also R22.1, U2.8 (GPIO6), U9.3; no longer R10.1, U2.36 (GPIO24), U4.3
- net S4: now also R10.1, U2.36 (GPIO24), U4.3; no longer R22.1, U2.8 (GPIO6), U9.3

Commit message: PCB modified and generated another design with the button
Parts:
- removed SW10, SW2, SW4, SW5, SW6, SW7, SW8, SW9: SW_Push, Design:Button, symbol Switch:SW_Push
- added J3, J4: (no value), symbol Connector_Generic:Conn_01x08
- BT4: value Battery_Cell -> (none); footprint Connector_PinHeader_2.54mm:PinHeader_1x02_P2.54mm_Vertical -> (none)
- BZ1: value Buzzer -> (none); footprint Connector_PinHeader_2.54mm:PinHeader_1x02_P2.54mm_Vertical -> (none)
- C1, C3: value 27pF -> (none); footprint Capacitor_SMD:C_0603_1608Metric -> (none)
- C10, C11, C12, C13, C14, C15, C16, C5, C6, C8, C9: value 100nF -> (none); footprint Capacitor_SMD:C_0402_1005Metric_Pad0.74x0.62mm_HandSolder -> (none)
- C2: value 0.1uF -> (none); footprint Capacitor_SMD:C_0402_1005Metric_Pad0.74x0.62mm_HandSolder -> (none)
- C20: value 47uF -> (none); footprint Capacitor_SMD:C_0603_1608Metric -> (none)
- C21, C22, C4, C7: value 1uF -> (none); footprint Capacitor_SMD:C_0603_1608Metric -> (none)
- C23, C24: value 220pF -> (none); footprint Capacitor_SMD:C_0603_1608Metric -> (none)
- C25, C26, C27: value 10uF -> (none); footprint Capacitor_SMD:C_0402_1005Metric_Pad0.74x0.62mm_HandSolder -> (none)
- C29: value 100nF -> (none); footprint Capacitor_SMD:C_0402_1005Metric -> (none)
- D1: value MBR120 -> (none); footprint Design:SODFL3616X98N -> (none)
- D2: value LED -> (none); footprint Capacitor_SMD:C_0603_1608Metric -> (none)
- F1: value 0.5A -> (none); footprint Fuse:Fuse_0805_2012Metric -> (none)
- J1: value Micro_SD_Card_Det -> (none); footprint Design:1140084168 -> (none)
- J2: value Conn_01x04_Female -> (none); footprint Connector_PinHeader_2.54mm:PinHeader_1x04_P2.54mm_Vertical -> (none)
- P1: value USB_C_Plug_USB2.0 -> (none); footprint Connectors:C393939 -> (none)
- Q1: value DMG3415U-7 -> (none); footprint Package_TO_SOT_SMD:SOT-23 -> (none)
- R1: value 1K -> (none); footprint Resistor_SMD:R_0603_1608Metric -> (none)
- R10, R11, R12, R22: value 10K -> (none); footprint Capacitor_SMD:C_0603_1608Metric -> (none)
- R13: value 1.8K -> (none); footprint Resistor_SMD:R_0603_1608Metric -> (none)
- R14, R15, R9: value 100 -> (none); footprint Resistor_SMD:R_0603_1608Metric -> (none)
- R16: value 10K -> (none); footprint Resistor_SMD:R_0603_1608Metric -> (none)
- R17, R23: value 100K -> (none); footprint Resistor_SMD:R_0603_1608Metric -> (none)
- R18, R19: value 5k1 -> (none); footprint Resistor_SMD:R_0603_1608Metric -> (none)
- R2, R3: value 27 -> (none); footprint Resistor_SMD:R_0603_1608Metric -> (none)
- R20: value 330 -> (none); footprint Resistor_SMD:R_0603_1608Metric -> (none)
- R21, R4, R6, R7: value 100 -> (none); footprint Capacitor_SMD:C_0603_1608Metric -> (none)
- R5: value 4K7 -> (none); footprint Resistor_SMD:R_0603_1608Metric -> (none)
- R8: value 220 -> (none); footprint Resistor_SMD:R_0603_1608Metric -> (none)
- SW1: value SW_DPDT_x2 -> (none); footprint Design:OS102011MA1QN1 -> (none)
- SW11: value SW_DPDT_x2 -> (none); footprint Design:7829H-1-051LF -> (none)
- SW12: value RESET -> (none); footprint Button_Switch_SMD:SW_SPST_TL3342 -> (none)
- SW13: value ON -> (none); footprint Design:OS102011MA1QN1 -> (none)
- SW14: value VOL -> (none); footprint Button_Switch_SMD:SW_SPST_TL3342 -> (none)
- SW15: value BOOT -> (none); footprint Button_Switch_SMD:SW_SPST_TL3342 -> (none)
- SW3: value REC -> (none); footprint Button_Switch_SMD:SW_SPST_TL3342 -> (none)
- U1: value SPH0641LM4H -> (none); footprint Sensors:MIC_SPH0641LM4H-1 -> (none)
- U10: value MCP4018-xxxxLT -> (none); footprint Design:SOT65P210X110-6N -> (none)
- U2: value RP2040 -> (none); footprint badge_pwnCon:RP2040-QFN-56 -> (none)
- U3, U4, U5, U9: value QRE1113 -> (none); footprint Design:QRE1113 -> (none)
- U6: value W25Q80DVSSIG -> (none); footprint Design:SOIC127P798X216-8N -> (none)
- U7: value PAM8302AASCR -> (none); footprint Package_SO:MSOP-8_3x3mm_P0.65mm -> (none)
- U8: value AP2112K-3.3 -> (none); footprint Package_TO_SOT_SMD:SOT-23-5 -> (none)
- Y1: value 12Mhz -> (none); footprint Crystal:Crystal_SMD_HC49-SD -> (none)
Connections:
- net D0: now also J3.3 (Pin_3)
- net D1: now also J3.7 (Pin_7)
- net D2: now also J4.5 (Pin_5)
- net D3: now also J3.5 (Pin_5)
- net D4: now also J4.3 (Pin_3)
- net D5: now also J3.1 (Pin_1)
- net D6: now also J4.1 (Pin_1)
- net D7: now also J4.7 (Pin_7)
- net GND: now also J3.2 (Pin_2), J3.4 (Pin_4), J3.6 (Pin_6), J3.8 (Pin_8), J4.2 (Pin_2), J4.4 (Pin_4), J4.6 (Pin_6), J4.8 (Pin_8)

Commit message: Update button and Kicad7
Parts:
- removed J3, J4: (no value), symbol Connector_Generic:Conn_01x08
- added J3, J5: Conn_01x05, symbol Connector_Generic:Conn_01x05
- BT4: value (none) -> Battery_Cell; footprint (none) -> Connector_PinHeader_2.54mm:PinHeader_1x02_P2.54mm_Vertical
- BZ1: value (none) -> Buzzer; footprint (none) -> Connector_PinHeader_2.54mm:PinHeader_1x02_P2.54mm_Vertical
- C1, C3: value (none) -> 27pF; footprint (none) -> Capacitor_SMD:C_0603_1608Metric
- C10, C11, C12, C13, C14, C15, C16, C5, C6, C8, C9: value (none) -> 100nF; footprint (none) -> Capacitor_SMD:C_0402_1005Metric_Pad0.74x0.62mm_HandSolder
- C2: value (none) -> 0.1uF; footprint (none) -> Capacitor_SMD:C_0402_1005Metric_Pad0.74x0.62mm_HandSolder
- C20: value (none) -> 47uF; footprint (none) -> Capacitor_SMD:C_0603_1608Metric
- C21, C22, C4, C7: value (none) -> 1uF; footprint (none) -> Capacitor_SMD:C_0603_1608Metric
- C23, C24: value (none) -> 220pF; footprint (none) -> Capacitor_SMD:C_0603_1608Metric
- C25, C26, C27: value (none) -> 10uF; footprint (none) -> Capacitor_SMD:C_0402_1005Metric_Pad0.74x0.62mm_HandSolder
- C29: value (none) -> 100nF; footprint (none) -> Capacitor_SMD:C_0402_1005Metric
- D1: value (none) -> MBR120; footprint (none) -> Design:SODFL3616X98N
- D2: value (none) -> LED; footprint (none) -> Capacitor_SMD:C_0603_1608Metric
- F1: value (none) -> 0.5A; footprint (none) -> Fuse:Fuse_0805_2012Metric
- J1: value (none) -> Micro_SD_Card_Det; footprint (none) -> Design:1140084168
- J2: value (none) -> Conn_01x04_Female; footprint (none) -> Connector_PinHeader_2.54mm:PinHeader_1x04_P2.54mm_Vertical
- P1: value (none) -> USB_C_Plug_USB2.0; footprint (none) -> Connectors:C393939
- Q1: value (none) -> DMG3415U-7; footprint (none) -> Package_TO_SOT_SMD:SOT-23
- R1: value (none) -> 1K; footprint (none) -> Resistor_SMD:R_0603_1608Metric
- R10, R11, R12, R22: value (none) -> 10K; footprint (none) -> Capacitor_SMD:C_0603_1608Metric
- R13: value (none) -> 1.8K; footprint (none) -> Resistor_SMD:R_0603_1608Metric
- R14, R15, R9: value (none) -> 100; footprint (none) -> Resistor_SMD:R_0603_1608Metric
- R16: value (none) -> 10K; footprint (none) -> Resistor_SMD:R_0603_1608Metric
- R17, R23: value (none) -> 100K; footprint (none) -> Resistor_SMD:R_0603_1608Metric
- R18, R19: value (none) -> 5k1; footprint (none) -> Resistor_SMD:R_0603_1608Metric
- R2, R3: value (none) -> 27; footprint (none) -> Resistor_SMD:R_0603_1608Metric
- R20: value (none) -> 330; footprint (none) -> Resistor_SMD:R_0603_1608Metric
- R21, R4, R6, R7: value (none) -> 100; footprint (none) -> Capacitor_SMD:C_0603_1608Metric
- R5: value (none) -> 4K7; footprint (none) -> Resistor_SMD:R_0603_1608Metric
- R8: value (none) -> 220; footprint (none) -> Resistor_SMD:R_0603_1608Metric
- SW1: value (none) -> SW_DPDT_x2; footprint (none) -> Design:OS102011MA1QN1
- SW11: value (none) -> SW_DPDT_x2; footprint (none) -> Design:7829H-1-051LF
- SW12: value (none) -> RESET; footprint (none) -> Button_Switch_SMD:SW_SPST_TL3342
- SW13: value (none) -> ON; footprint (none) -> Design:OS102011MA1QN1
- SW14: value (none) -> VOL; footprint (none) -> Button_Switch_SMD:SW_SPST_TL3342
- SW15: value (none) -> BOOT; footprint (none) -> Button_Switch_SMD:SW_SPST_TL3342
- SW3: value (none) -> REC; footprint (none) -> Button_Switch_SMD:SW_SPST_TL3342
- U1: value (none) -> SPH0641LM4H; footprint (none) -> Sensors:MIC_SPH0641LM4H-1
- U10: value (none) -> MCP4018-xxxxLT; footprint (none) -> Design:SOT65P210X110-6N
- U2: value (none) -> RP2040; footprint (none) -> badge_pwnCon:RP2040-QFN-56
- U3, U4, U5, U9: value (none) -> QRE1113; footprint (none) -> Design:QRE1113
- U6: value (none) -> W25Q80DVSSIG; footprint (none) -> Design:SOIC127P798X216-8N
- U7: value (none) -> PAM8302AASCR; footprint (none) -> Package_SO:MSOP-8_3x3mm_P0.65mm
- U8: value (none) -> AP2112K-3.3; footprint (none) -> Package_TO_SOT_SMD:SOT-23-5
- Y1: value (none) -> 12Mhz; footprint (none) -> Crystal:Crystal_SMD_HC49-SD
Connections:
- net D0: now also J5.3 (Pin_3)
- net D1: now also J5.5 (Pin_5)
- net D2: now also J3.3 (Pin_3)
- net D3: now also J5.4 (Pin_4)
- net D4: now also J3.2 (Pin_2)
- net D5: now also J5.2 (Pin_2)
- net D6: now also J3.1 (Pin_1)
- net D7: now also J3.4 (Pin_4)
- net GND: now also J5.1 (Pin_1)
- net D8: now reaches U2.9 (GPIO7)
- net D8: now also J3.5 (Pin_5)
- no-connect marks 5 -> 4
