File: hardware/DesignLab.kicad_pcb (KiCad board)
At the start: 2 copper layers, 0 parts

Commit message: Assigned footprints
Other:
- net class Default removed
Changed lines of the file:
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@@
-(kicad_pcb (version 20171130) (host pcbnew "(5.1.9-0-10_14)")
+(kicad_pcb (version 20211014) (generator pcbnew)
   (general
     (thickness 1.6)
-    (drawings 0)
-    (tracks 0)
-    (zones 0)
-    (modules 0)
-    (nets 1)
   )
-  (page A4)
+  (paper "A4")
   (layers
-    (0 Top signal)
-    (31 Bottom signal)
-    (32 B.Adhes user)
-    (33 F.Adhes user)
-    (34 B.Paste user)
-    (35 F.Paste user)
-    (36 B.SilkS user)
-    (37 F.SilkS user)
-    (38 B.Mask user)
-    (39 F.Mask user)
-    (40 Dwgs.User user)
-    (41 Cmts.User user)
-    (42 Eco1.User user)
-    (43 Eco2.User user)
-    (44 Edge.Cuts user)
-    (45 Margin user)
-    (46 B.CrtYd user)
-    (47 F.CrtYd user)
-    (48 B.Fab user)
-    (49 F.Fab user)
+    (0 "F.Cu" signal "Top")
+    (31 "B.Cu" signal "Bottom")
+    (32 "B.Adhes" user "B.Adhesive")
+    (33 "F.Adhes" user "F.Adhesive")
+    (34 "B.Paste" user)
+    (35 "F.Paste" user)
+    (36 "B.SilkS" user "B.Silkscreen")
+    (37 "F.SilkS" user "F.Silkscreen")
+    (38 "B.Mask" user)
+    (39 "F.Mask" user)
+    (40 "Dwgs.User" user "User.Drawings")
+    (41 "Cmts.User" user "User.Comments")
+    (42 "Eco1.User" user "User.Eco1")
+    (43 "Eco2.User" user "User.Eco2")
+    (44 "Edge.Cuts" user)
+    (45 "Margin" user)
+    (46 "B.CrtYd" user "B.Courtyard")
+    (47 "F.CrtYd" user "F.Courtyard")
+    (48 "B.Fab" user)
+    (49 "F.Fab" user)
   )
   (setup
-    (last_trace_width 0.2)
-    (user_trace_width 0.2)
-    (user_trace_width 0.25)
-    (user_trace_width 0.3)
-    (user_trace_width 0.4)
-    (user_trace_width 0.5)
-    (user_trace_width 0.6)
-    (user_trace_width 1)
-    (trace_clearance 0.2)
-    (zone_clearance 0.508)
-    (zone_45_only no)
-    (trace_min 0.1524)
-    (via_size 0.6)
-    (via_drill 0.3)
-    (via_min_size 0.6)
-    (via_min_drill 0.3)
-    (user_via 0.6 0.3)
-    (user_via 0.8 0.4)
-    (uvia_size 0.6)
-    (uvia_drill 0.3)
-    (uvias_allowed no)
-    (uvia_min_size 0.2)
-    (uvia_min_drill 0.1)
-    (edge_width 0.15)
-    (segment_width 0.2)
-    (pcb_text_width 0.3)
-    (pcb_text_size 1.5 1.5)
-    (mod_edge_width 0.15)
-    (mod_text_size 1 1)
-    (mod_text_width 0.15)
-    (pad_size 1.524 1.524)
-    (pad_drill 0.762)
     (pad_to_mask_clearance 0)
-    (aux_axis_origin 0 0)
-    (visible_elements 7FFFFFFF)
     (pcbplotparams
-      (layerselection 0x010fc_ffffffff)
+      (layerselection 0x00010fc_ffffffff)
+      (disableapertmacros false)
       (usegerberextensions false)
       (usegerberattributes false)
       (usegerberadvancedattributes false)
       (creategerberjobfile false)
+      (svguseinch false)
+      (svgprecision 6)
       (excludeedgelayer true)
-      (linewidth 0.100000)
       (plotframeref false)
       (viasonmask false)
@@
       (hpglpenspeed 20)
       (hpglpendiameter 15.000000)
+      (dxfpolygonmode true)
+      (dxfimperialunits true)
+      (dxfusepcbnewfont true)
       (psnegative false)
       (psa4output false)
@@
       (plotvalue true)
       (plotinvisibletext false)
-      (padsonsilk false)
+      (sketchpadsonfab false)
       (subtractmaskfromsilk false)
       (outputformat 1)
@@
       (drillshape 1)
       (scaleselection 1)
-      (outputdirectory ""))
+      (outputdirectory "")
+    )
   )
   (net 0 "")
-  (net_class Default "This is the default net class."
-    (clearance 0.2)
-    (trace_width 0.2)
-    (via_dia 0.6)
-    (via_drill 0.3)
-    (uvia_dia 0.6)
-    (uvia_drill 0.3)
-    (diff_pair_width 0.1524)
-    (diff_pair_gap 0.1524)
-  )
 )

Commit message: PCB design proposal
Parts:
- added BT4: Battery_Cell, Design:2477, F.Cu at (182.8, 202.5)
- added BZ1: Buzzer, Connector_PinHeader_2.54mm:PinHeader_1x02_P2.54mm_Vertical, F.Cu at (271.4, 165.2)
- added C1: 27pF, Capacitor_SMD:C_0603_1608Metric, F.Cu at (196.1, 167.8)
- added C10: 100nF, Capacitor_SMD:C_0402_1005Metric_Pad0.74x0.62mm_HandSolder, F.Cu at (186.8, 182.2)
- added C11: 100nF, Capacitor_SMD:C_0402_1005Metric_Pad0.74x0.62mm_HandSolder, F.Cu at (194.4, 190.1)
- added C12: 100nF, Capacitor_SMD:C_0402_1005Metric_Pad0.74x0.62mm_HandSolder, F.Cu at (188.6, 190.1)
- added C13: 100nF, Capacitor_SMD:C_0402_1005Metric_Pad0.74x0.62mm_HandSolder, F.Cu at (186.8, 185.8)
- added C14: 100nF, Capacitor_SMD:C_0402_1005Metric_Pad0.74x0.62mm_HandSolder, F.Cu at (186.8, 183.2)
- added C15: 100nF, Capacitor_SMD:C_0402_1005Metric_Pad0.74x0.62mm_HandSolder, F.Cu at (193.2, 197.0)
- added C16: 100nF, Capacitor_SMD:C_0402_1005Metric_Pad0.74x0.62mm_HandSolder, F.Cu at (237.6, 172.4)
- added C17: 10nF, Capacitor_SMD:C_0603_1608Metric, F.Cu at (152.1, 157.7)
- added C18: 10nF, Capacitor_SMD:C_0603_1608Metric, F.Cu at (223.5, 157.9)
- added C19: 10nF, Capacitor_SMD:C_0603_1608Metric, F.Cu at (244.2, 156.3)
- added C2: 0.1uF, Capacitor_SMD:C_0402_1005Metric_Pad0.74x0.62mm_HandSolder, F.Cu at (175.8, 182.8)
- added C20: 47uF, Capacitor_SMD:C_0603_1608Metric, F.Cu at (240.6, 172.4)
- added C21: 1uF, Capacitor_SMD:C_0603_1608Metric, F.Cu at (246.5, 167.2)
- added C22: 1uF, Capacitor_SMD:C_0603_1608Metric, F.Cu at (246.4, 164.2)
- added C23: 220pF, Capacitor_SMD:C_0603_1608Metric, F.Cu at (263.7, 164.9)
- added C24: 220pF, Capacitor_SMD:C_0603_1608Metric, F.Cu at (263.8, 168.4)
- added C25: 10uF, Capacitor_SMD:C_0402_1005Metric_Pad0.74x0.62mm_HandSolder, F.Cu at (255.8, 161.9)
- added C26: 10uF, Capacitor_SMD:C_0402_1005Metric_Pad0.74x0.62mm_HandSolder, F.Cu at (147.0, 192.4)
- added C27: 10uF, Capacitor_SMD:C_0402_1005Metric_Pad0.74x0.62mm_HandSolder, F.Cu at (156.3, 190.6)
- added C28: 10nF, Capacitor_SMD:C_0603_1608Metric, F.Cu at (186.1, 159.0)
- added C29: 100nF, Capacitor_SMD:C_0402_1005Metric, F.Cu at (141.1, 183.7)
- added C3: 27pF, Capacitor_SMD:C_0603_1608Metric, F.Cu at (185.9, 167.8)
- added C4: 1uF, Capacitor_SMD:C_0603_1608Metric, F.Cu at (200.1, 184.6)
- added C5: 100nF, Capacitor_SMD:C_0402_1005Metric_Pad0.74x0.62mm_HandSolder, F.Cu at (189.5, 190.1)
- added C6: 100nF, Capacitor_SMD:C_0402_1005Metric_Pad0.74x0.62mm_HandSolder, F.Cu at (194.6, 176.5)
- added C7: 1uF, Capacitor_SMD:C_0603_1608Metric, F.Cu at (193.3, 176.1)
- added C8: 100nF, Capacitor_SMD:C_0402_1005Metric_Pad0.74x0.62mm_HandSolder, F.Cu at (199.7, 182.2)
- added C9: 100nF, Capacitor_SMD:C_0402_1005Metric_Pad0.74x0.62mm_HandSolder, F.Cu at (190.4, 190.1)
- added D1: MBR120, Design:SODFL3616X98N, F.Cu at (141.2, 197.2)
- added D2: LED, Capacitor_SMD:C_0603_1608Metric, F.Cu at (183.1, 196.0)
- added F1: 0.5A, Fuse:Fuse_0805_2012Metric, F.Cu at (137.7, 196.1)
- added J1: Micro_SD_Card_Det, Design:1140084168, F.Cu at (131.8, 183.8)
- added J2: Conn_01x04_Female, Connector_PinHeader_2.54mm:PinHeader_1x04_P2.54mm_Vertical, F.Cu at (179.9, 209.1)
- added P1: USB_C_Plug_USB2.0, Connectors:C393939, F.Cu at (131.2, 200.2)
- added Q1: DMG3415U-7, Package_TO_SOT_SMD:SOT-23, F.Cu at (145.1, 197.2)
- added R1: 1K, Resistor_SMD:R_0603_1608Metric, F.Cu at (191.8, 176.1)
- added R10: 220, Capacitor_SMD:C_0603_1608Metric, F.Cu at (152.1, 159.2)
- added R11: 220, Capacitor_SMD:C_0603_1608Metric, F.Cu at (223.5, 159.4)
- added R12: 220, Capacitor_SMD:C_0603_1608Metric, F.Cu at (244.2, 157.8)
- added R13: 1.8K, Resistor_SMD:R_0603_1608Metric, F.Cu at (242.1, 172.4)
- added R14: 100, Resistor_SMD:R_0603_1608Metric, F.Cu at (250.4, 167.2)
- added R15: 100, Resistor_SMD:R_0603_1608Metric, F.Cu at (250.4, 165.1)
- added R16: 10K, Resistor_SMD:R_0603_1608Metric, F.Cu at (255.8, 171.7)
- added R17: 100K, Resistor_SMD:R_0603_1608Metric, F.Cu at (142.0, 193.6)
- added R18: 5k1, Resistor_SMD:R_0603_1608Metric, F.Cu at (137.4, 199.8)
- added R19: 5k1, Resistor_SMD:R_0603_1608Metric, F.Cu at (137.4, 203.2)
- added R2: 27, Resistor_SMD:R_0603_1608Metric, F.Cu at (193.2, 190.5)
- added R20: 330, Resistor_SMD:R_0603_1608Metric, F.Cu at (183.1, 197.5)
- added R21: 100, Capacitor_SMD:C_0603_1608Metric, F.Cu at (186.1, 157.5)
- added R22: 220, Capacitor_SMD:C_0603_1608Metric, F.Cu at (186.1, 160.5)
- added R23: 100K, Resistor_SMD:R_0603_1608Metric, F.Cu at (141.7, 186.1)
- added R3: 27, Resistor_SMD:R_0603_1608Metric, F.Cu at (191.7, 190.5)
- added R4: 100, Capacitor_SMD:C_0603_1608Metric, F.Cu at (152.1, 156.2)
- added R5: 4K7, Resistor_SMD:R_0603_1608Metric, F.Cu at (202.9, 199.2)
- added R6: 100, Capacitor_SMD:C_0603_1608Metric, F.Cu at (223.5, 156.5)
- added R7: 100, Capacitor_SMD:C_0603_1608Metric, F.Cu at (244.2, 159.3)
- added R8: 220, Resistor_SMD:R_0603_1608Metric, F.Cu at (236.1, 172.4)
- added R9: 100, Resistor_SMD:R_0603_1608Metric, F.Cu at (239.1, 172.4)
- added SW1: SW_DPDT_x2, Design:OS102011MA1QN1, F.Cu at (259.2, 188.8)
- added SW10: Button, Design:EVQPLFA08, F.Cu at (236.8, 98.8)
- added SW11: Button, Design:EVQPLFA08, F.Cu at (123.7, 138.6)
- added SW12: RESET, Button_Switch_SMD:SW_SPST_TL3342, F.Cu at (158.3, 167.6)
- added SW13: ON, Design:OS102011MA1QN1, F.Cu at (126.8, 167.1)
- added SW14: VOL, Button_Switch_SMD:SW_SPST_TL3342, F.Cu at (229.4, 204.4)
- added SW15: BOOT, Button_Switch_SMD:SW_SPST_TL3342, F.Cu at (158.4, 205.1)
- added SW2: SW_DPDT_x2, Design:OS102011MA1QN1, F.Cu at (229.6, 188.6)
- added SW3: REC, Button_Switch_SMD:SW_SPST_TL3342, F.Cu at (259.2, 204.4)
- added SW4: Button, Design:EVQPLFA08, F.Cu at (161.8, 98.8)
- added SW5: Button, Design:EVQPLFA08, F.Cu at (124.3, 58.8)
- added SW6: Button, Design:EVQPLFA08, F.Cu at (274.3, 138.9)
- added SW7: Button, Design:EVQPLFA08, F.Cu at (274.2, 58.8)
- added SW8: Button, Design:EVQPLFA08, F.Cu at (199.3, 58.8)
- added SW9: Button, Design:EVQPLFA08, F.Cu at (199.3, 138.8)
- added U1: SPH0641LM4H, Sensors:MIC_SPH0641LM4H-1, F.Cu at (179.5, 184.0)
- added U10: MCP4018-xxxxLT, Design:SOT65P210X110-6N, F.Cu at (241.4, 165.6)
- added U2: RP2040, badge_pwnCon:RP2040-QFN-56, F.Cu at (193.2, 183.2)
- added U3: QRE1113, Design:QRE1113, F.Cu at (147.3, 156.7)
- added U4: QRE1113, Design:QRE1113, F.Cu at (219.4, 157.2)
- added U5: QRE1113, Design:QRE1113, F.Cu at (249.6, 158.8)
- added U6: AT25SF128A, Design:SOIC127P798X216-8N, F.Cu at (200.2, 195.1)
- added U7: PAM8302AAD, Package_SO:MSOP-8_3x3mm_P0.65mm, F.Cu at (255.9, 166.7)
- added U8: AP2112K-3.3, Package_TO_SOT_SMD:SOT-23-5, F.Cu at (151.7, 191.5)
- added U9: QRE1113, Design:QRE1113, F.Cu at (181.3, 157.4)
- added Y1: 12Mhz, Crystal:Crystal_SMD_HC49-SD, F.Cu at (190.9, 171.9)

Commit message: More PCB design proposal
Parts:
- BT4, J1, J2, P1, SW12, SW15: moved to B.Cu
- moved SW15 87.9 mm to (236.7, 165.1), turned to 180 degrees
- moved SW12 78.4 mm to (236.5, 173.2), turned to 180 degrees
- moved U1 63.7 mm to (124.0, 152.7), turned to 180 degrees
- moved C2 55.4 mm to (128.5, 153.9), turned to 0 degrees
- moved J2 50.4 mm to (154.4, 165.6), turned to 180 degrees
- moved BT4 18.4 mm to (201.2, 203.0)
- moved C28 17.0 mm to (185.2, 142.0)
- moved R10 17.0 mm to (151.2, 142.2)
- moved R12 17.0 mm to (243.3, 140.8)
- moved R21 17.0 mm to (185.2, 140.5)
- moved R22 17.0 mm to (185.2, 143.5)
- moved R6 17.0 mm to (222.6, 139.5)
- moved R7 17.0 mm to (243.3, 142.3)
- moved U3 17.0 mm to (146.4, 139.7)
- moved U5 17.0 mm to (248.7, 141.8)
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Other:
- board outline added: 161 x 180.3 mm
- board text added: "LANG"
- board text added: "MIC"
- board text added: "ON/OFF"
- board text added: "REC"
- board text added: "VOL"
- board text added: "WORDS"

Commit message: Update foorplan
Parts:
- J1, P1: moved to F.Cu
- SW3: moved to B.Cu
- moved C2 145.8 mm to (274.3, 151.4)
- moved U1 145.8 mm to (269.8, 150.3)
- moved BT4 137.4 mm to (67.1, 173.0)
- moved SW14 74.1 mm to (165.9, 186.2)
- moved J2 73.5 mm to (227.8, 169.2), turned to 0 degrees
- moved SW3 51.7 mm to (236.7, 155.4)
- moved C27 34.0 mm to (178.8, 165.2)
- moved C29 34.0 mm to (163.6, 158.3)
- moved F1 34.0 mm to (160.2, 170.7)
- moved R19 34.0 mm to (160.0, 177.8)
- moved C26 34.0 mm to (169.6, 167.1)
- moved D1 34.0 mm to (163.7, 171.8)
- moved Q1 34.0 mm to (167.7, 171.9)
- moved R17 34.0 mm to (164.6, 168.2)
- moved R18 34.0 mm to (160.0, 174.5)
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
Commit message: PCB layout and .step file
Parts:
- BT4: footprint Design:2477 -> Connector_PinHeader_2.54mm:PinHeader_1x02_P2.54mm_Vertical
- moved BT4 56.0 mm to (122.1, 162.7), turned to 180 degrees
- moved F1 39.1 mm to (132.7, 198.5)
- moved D1 38.3 mm to (136.2, 198.4)
- moved Q1 38.3 mm to (140.2, 198.5)
- moved R17 38.3 mm to (137.1, 194.8)
- moved R18 37.7 mm to (132.5, 200.2)
- moved R19 37.5 mm to (132.5, 203.2)
- moved C29 34.5 mm to (136.5, 179.7)
- moved R23 34.5 mm to (137.1, 182.1)
- moved U8 31.1 mm to (149.8, 185.3)
- moved C27 31.1 mm to (154.4, 184.4)
- moved C26 30.8 mm to (145.6, 186.3)
- moved SW13 9.52 mm to (146.2, 193.7)
- moved SW14 7.26 mm to (165.1, 193.4)
- moved R8 5.72 mm to (241.8, 171.5)
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Other:
- outline, holes or cut-outs redrawn

Commit message: new size
Parts:
- moved SW11 24.6 mm to (146.8, 118.4)
- moved SW5 21.3 mm to (145.8, 47.0)
- moved SW6 10.8 mm to (268.7, 118.4)
- moved C23 10.1 mm to (277.2, 169.0)
- moved R13 10.1 mm to (256.9, 175.7)
- moved R16 10.1 mm to (270.4, 175.7)
- moved C21 10.1 mm to (261.1, 171.3)
- moved C16 10.1 mm to (252.5, 175.7)
- moved C20 10.1 mm to (255.4, 175.7)
- moved R8 10.1 mm to (251.0, 175.7)
- moved R9 10.1 mm to (253.9, 175.7)
- moved BZ1 10.1 mm to (285.5, 169.5)
- moved R14 10.1 mm to (265.0, 171.3)
- moved U10 10.1 mm to (256.3, 169.9)
- moved C22 10.1 mm to (261.0, 168.2)
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Other:
- board size 161 x 180.3 mm -> 169.9 x 180.3 mm
- board text added: "Battery"

Commit message: move buttons
Parts:
- moved D2 13.4 mm to (194.3, 191.7)
- moved R20 13.4 mm to (194.3, 193.2)
- moved C1 13.4 mm to (209.1, 164.6)
- moved C10 13.4 mm to (199.8, 179.1)
- moved C11 13.4 mm to (207.4, 187.0)
- moved C12 13.4 mm to (201.6, 187.0)
- moved C13 13.4 mm to (199.8, 182.7)
- moved C14 13.4 mm to (199.8, 180.1)
- moved C15 13.4 mm to (206.2, 193.9)
- moved C3 13.4 mm to (198.9, 164.7)
- moved C4 13.4 mm to (213.1, 181.5)
- moved C5 13.4 mm to (202.5, 187.0)
- moved C6 13.4 mm to (207.6, 173.4)
- moved C7 13.4 mm to (206.3, 173.0)
- moved C8 13.4 mm to (212.7, 179.1)
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