File: hardware/Buttons/LeftButtonsDesignLab/LeftButtonsDesignLab.kicad_pcb (KiCad board)
At the start: 2 copper layers, 26 x 105 mm, 5 parts, among them J1 Conn_01x04, J2 Conn_01x01, SW1 SW_Push, SW2 SW_Push, SW3 SW_Push

Commit message: labels buttons
Other:
- board text added: "D0"
- board text added: "D3"
- board text added: "D6"
- board text added: "GND"
