File: hardware/Buttons/LeftButtonsDesignLab/LeftButtonsDesignLab.kicad_pcb (KiCad board)
At the start: 2 copper layers, 26 x 105 mm, 5 parts, among them J1 Conn_01x04, J2 Conn_01x01, SW1 SW_Push, SW2 SW_Push, SW3 SW_Push

Commit message: Update all PCB and schematics
Parts:
- removed J2: Conn_01x01, Connector_PinHeader_2.54mm:PinHeader_1x01_P2.54mm_Vertical
- J1: footprint Connector_PinHeader_2.54mm:PinHeader_1x04_P2.54mm_Vertical -> Design:JST_S4B-PH-K-S_LF__SN_; moved to B.Cu
- moved J1 3.91 mm to (132.7, 134.5), turned to -90 degrees
Connections:
- J1 pad 1: /GND -> /D0
- J1 pad 2: /D6 -> /D3
- J1 pad 3: /D3 -> /D6
- J1 pad 4: /D0 -> /GND
Routing:
- net /D6: track 29.1 -> 28.0 mm
- net /D3: track 63.8 -> 63.3 mm
Other:
- board size 26 x 105 mm -> 29.8 x 105 mm
