File: hardware/Buttons/RightButtonsDesignLab/RightButtonsDesignLab.kicad_pcb (KiCad board)
At the start: 2 copper layers, 26 x 105 mm, 5 parts, among them J1 Conn_01x03, J2 Conn_01x01, SW1 SW_Push, SW2 SW_Push, SW3 SW_Push

Commit message: Update all PCB and schematics
Parts:
- removed J2: Conn_01x01, Connector_PinHeader_2.54mm:PinHeader_1x01_P2.54mm_Vertical
- J1: value Conn_01x03 -> Conn_01x04; footprint Connector_PinHeader_2.54mm:PinHeader_1x03_P2.54mm_Vertical -> Design:JST_S4B-PH-K-S_LF__SN_; moved to B.Cu
- moved J1 2.87 mm to (123.9, 136.8), turned to 90 degrees
Routing:
- net /D8: track 35.0 -> 34.2 mm
- net /GND: vias 0 -> 1
Other:
- board size 26 x 105 mm -> 30 x 105 mm
- board text removed: "GND"
