File: hardware/Buttons/RightButtonsDesignLab/RightButtonsDesignLab.kicad_pcb (KiCad board)
At the start: 2 copper layers, 30 x 105 mm, 4 parts, among them J1 Conn_01x04, SW1 SW_Push, SW2 SW_Push, SW3 SW_Push

Commit message: Update PCB
Parts:
- moved J1 15.4 mm to (139.3, 136.7), turned to -90 degrees
- turned SW3 to -90 degrees
Connections:
- J1 pad 1: /D8 -> /GND
- J1 pad 2: /D5 -> /D2
- J1 pad 3: /D2 -> /D5
- J1 pad 4: /GND -> /D8
Routing:
- net /D5: track 65.4 -> 60.6 mm, vias 0 -> 1
- net /D2: track 91.4 -> 95.4 mm
- net /GND: vias 1 -> 0
Other:
- board size 30 x 105 mm -> 26 x 105 mm

Commit message: Update PCB of buttons
Other:
- board size 26 x 105 mm -> 22 x 105 mm

Commit message: .steps updated
Changed lines of the file:
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@@
   (gr_line (start 147.61 100.23) (end 147.61 80.23)
     (stroke (width 0.1) (type solid)) (layer "Edge.Cuts"))
-  (gr_line (start 137.59 37.72) (end 125.59 37.72)
+  (gr_line (start 137.61 37.72) (end 125.61 37.72)
     (stroke (width 0.1) (type solid)) (layer "Edge.Cuts"))
   (gr_circle (center 131.63 41.805) (end 133.13 41.805)
@@
   (gr_line (start 145.62 130.73) (end 137.61 130.73)
     (stroke (width 0.1) (type solid)) (layer "Edge.Cuts"))
-  (gr_line (start 137.61 80.23) (end 137.61 37.73)
+  (gr_line (start 137.61 80.23) (end 137.61 37.72)
     (stroke (width 0.1) (type solid)) (layer "Edge.Cuts"))
   (gr_line (start 147.61 80.23) (end 137.61 80.23)

Commit message: Update label buttons
Other:
- board text added: "GND"
