File: hardware/Buttons/CenterButtonsDesignLab/CenterButtonsDesignLab.kicad_pcb (KiCad board)
At the start: 2 copper layers, 23 x 118 mm, 5 parts, among them J1 Conn_01x05, SW1 SW_Push, SW2 SW_Push, SW3 SW_Push, SW4 SW_Push

Commit message: Update PCB
Parts:
- moved J1 15.7 mm to (186.6, 136.8), turned to -90 degrees
- turned SW1 to 90 degrees
- turned SW3 to -90 degrees
- turned SW4 to 90 degrees
Connections:
- J1 pad 2: /D7 -> /D9
- J1 pad 3: /D4 -> /D1
- J1 pad 4: /D1 -> /D4
- J1 pad 5: /D9 -> /D7
Routing:
- net /D7: track 30.9 -> 29.5 mm
- net /D4: track 54.7 -> 54.1 mm
- net /D9: track 102.7 -> 102.1 mm
- net /GND: vias 0 -> 1
Other:
- outline, holes or cut-outs redrawn

Commit message: Update label buttons
Other:
- board text added: "D9"
- board text added: "GND"
